File: rev1/PCB/corne-xiao.kicad_sch (KiCad schematic)
At the start: 110 parts, among them J1 OLED, SW1 SW_PUSH, SW10 SW_PUSH, SW11 SW_PUSH, SW12 SW_PUSH, SW13 SW_PUSH, SW14 SW_PUSH, SW15 SW_PUSH, SW16 SW_PUSH, SW17 SW_PUSH, SW18 SW_PUSH, SW19 SW_PUSH, SW2 SW_PUSH, SW20 SW_PUSH, SW21 SW_PUSH, SW22 SW_PUSH, SW23 SW_PUSH, SW24 SW_PUSH, SW25 SW_PUSH, SW26 SW_PUSH, SW27 SW_PUSH, SW28 SW_PUSH, SW29 SW_PUSH, SW3 SW_PUSH, SW30 SW_PUSH, SW31 SW_PUSH, SW32 SW_PUSH, SW33 SW_PUSH, SW34 SW_PUSH, SW35 SW_PUSH, SW36 SW_PUSH, SW37 SW_PUSH, SW38 SW_PUSH, SW39 SW_PUSH, SW4 SW_PUSH, SW40 SW_PUSH, SW41 SW_PUSH, SW42 SW_PUSH, SW43 RotaryEncoder_Switch, SW44 RotaryEncoder_Switch, SW5 SW_PUSH, SW6 SW_PUSH, SW7 SW_PUSH, SW8 SW_PUSH, SW9 SW_PUSH, U1 xiao-ble, U2 xiao-ble

Commit message: Start
Parts:
- removed SW43, SW44: RotaryEncoder_Switch, fp:RotaryEncoder_Alps_EC11E-Switch_Vertical_H20mm-keebio_modified, symbol Device:RotaryEncoder_Switch
- SW1, SW10, SW11, SW12, SW13, SW14, SW15, SW16, SW17, SW18, SW19, SW2, SW20, SW22, SW23, SW24, SW25, SW26, SW27, SW28, SW29, SW3, SW30, SW31, SW32, SW33, SW34, SW35, SW36, SW37, SW38, SW39, SW4, SW40, SW41, SW5, SW6, SW7, SW8, SW9: footprint kbd:CherryMX_Hotswap -> keeb_switches:CPG1316S01D02_mikeholscher
- SW21, SW42: footprint kbd:CherryMX_Hotswap_1.5u -> keeb_switches:CPG1316S01D02_mikeholscher

Commit message: moar
Parts:
- removed D43, D44: D, kbd:D3_SMD_v2, symbol Device:D
- removed J1 (x2): OLED, fp:nice_view, symbol Connector_Generic:Conn_01x05
