File: rev1/PCB/corne-xiao.kicad_pcb (KiCad board)
At the start: 2 copper layers, 254.7 x 101.7 mm, 94 parts, among them SW1 SW_PUSH, SW10 SW_PUSH, SW11 SW_PUSH, SW12 SW_PUSH, SW13 SW_PUSH, SW14 SW_PUSH, SW15 SW_PUSH, SW16 SW_PUSH, SW17 SW_PUSH, SW18 SW_PUSH, SW19 SW_PUSH, SW2 SW_PUSH, SW20 SW_PUSH, SW21 SW_PUSH, SW22 SW_PUSH, SW23 SW_PUSH, SW24 SW_PUSH, SW25 SW_PUSH, SW26 SW_PUSH, SW27 SW_PUSH, SW28 SW_PUSH, SW29 SW_PUSH, SW3 SW_PUSH, SW30 SW_PUSH, SW31 SW_PUSH, SW32 SW_PUSH, SW33 SW_PUSH, SW34 SW_PUSH, SW35 SW_PUSH, SW36 SW_PUSH, SW37 SW_PUSH, SW38 SW_PUSH, SW39 SW_PUSH, SW4 SW_PUSH, SW40 SW_PUSH, SW41 SW_PUSH, SW42 SW_PUSH, SW5 SW_PUSH, SW6 SW_PUSH, SW7 SW_PUSH, SW8 SW_PUSH, SW9 SW_PUSH, U1 xiao-ble, U2 xiao-ble

Commit message: Backup
Parts:
- D1, D10, D11, D12, D13, D14, D15, D16, D17, D18, D19, D2, D20, D21, D22, D23, D24, D25, D26, D27, D28, D29, D3, D30, D31, D32, D33, D34, D35, D36, D37, D38, D39, D4, D40, D41, D42, D5, D6, D7, D8, D9: footprint kbd:D3_SMD_v2 -> ScottoKeebs_Components:Diode_SOD-123
- moved U1 1.05 mm to (136.1, 39.0)
- moved U2 1.05 mm to (163.4, 39.1)
- moved D20 0.71 mm to (109.7, 89.2)
- moved D13 0.70 mm to (31.6, 71.5)
- moved D7 0.70 mm to (31.6, 54.5)
- moved D4 0.68 mm to (82.6, 30.3)
- moved D16 0.68 mm to (82.6, 64.3)
- moved D10 0.68 mm to (82.6, 47.3)
- moved D6 0.67 mm to (116.6, 35.1)
- moved D18 0.67 mm to (116.6, 69.1)
- moved D5 0.65 mm to (99.6, 32.7)
- moved D11 0.65 mm to (99.6, 49.7)
- moved D17 0.65 mm to (99.6, 66.7)
- moved D2 0.64 mm to (48.6, 37.5)
- moved D8 0.64 mm to (48.6, 54.5)
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Routing:
- net unconnected-(PSW1-A-Pad1): track 59.1 -> 0.00 mm
- net ROW3_L: track 79.4 -> 103.0 mm, vias 2 -> 1
- net ROW0_L: track 91.5 -> 111.5 mm, vias 5 -> 0
- net COL4_R: track 108.6 -> 124.1 mm
- net COL1_L: track 155.7 -> 141.7 mm, vias 7 -> 5
- net ROW3_R: track 113.7 -> 124.5 mm, vias 1 -> 2
- net BAT+_L: track 66.7 -> 58.3 mm
- net COL3_R: track 131.4 -> 138.8 mm, vias 9 -> 7
- net GND: track 23.2 -> 30.2 mm
- net Net-(D9-A): track 6.86 -> 11.9 mm
- net ROW1_R: track 133.6 -> 138.5 mm
- net ROW0_R: track 122.7 -> 127.1 mm
- net COL5_L: track 75.9 -> 71.7 mm, vias 7 -> 5
- net COL4_L: track 147.4 -> 144.4 mm
- net VBAT_R: track 40.0 -> 42.9 mm
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Other:
- outline, holes or cut-outs redrawn
