File: rev1/PCB/corne-xiao-backups/backup/corne-xiao.kicad_pcb (KiCad board)
At the start: 2 copper layers, 254.7 x 101.7 mm, 94 parts, among them SW1 SW_PUSH, SW10 SW_PUSH, SW11 SW_PUSH, SW12 SW_PUSH, SW13 SW_PUSH, SW14 SW_PUSH, SW15 SW_PUSH, SW16 SW_PUSH, SW17 SW_PUSH, SW18 SW_PUSH, SW19 SW_PUSH, SW2 SW_PUSH, SW20 SW_PUSH, SW21 SW_PUSH, SW22 SW_PUSH, SW23 SW_PUSH, SW24 SW_PUSH, SW25 SW_PUSH, SW26 SW_PUSH, SW27 SW_PUSH, SW28 SW_PUSH, SW29 SW_PUSH, SW3 SW_PUSH, SW30 SW_PUSH, SW31 SW_PUSH, SW32 SW_PUSH, SW33 SW_PUSH, SW34 SW_PUSH, SW35 SW_PUSH, SW36 SW_PUSH, SW37 SW_PUSH, SW38 SW_PUSH, SW39 SW_PUSH, SW4 SW_PUSH, SW40 SW_PUSH, SW41 SW_PUSH, SW42 SW_PUSH, SW5 SW_PUSH, SW6 SW_PUSH, SW7 SW_PUSH, SW8 SW_PUSH, SW9 SW_PUSH, U1 xiao-ble, U2 xiao-ble

Commit message: Backup
Parts:
- moved U1 1.05 mm to (136.1, 40.1)
- moved U2 1.05 mm to (163.4, 40.2)
Routing:
- net unconnected-(PSW1-A-Pad1): track 0.00 -> 59.1 mm
- net ROW3_L: track 101.3 -> 79.4 mm, vias 1 -> 2
- net ROW0_L: track 110.9 -> 91.5 mm, vias 0 -> 5
- net COL1_L: track 137.7 -> 155.7 mm, vias 5 -> 7
- net COL4_R: track 124.1 -> 108.6 mm
- net ROW3_R: track 124.5 -> 113.7 mm, vias 2 -> 1
- net BAT+_L: track 58.3 -> 66.7 mm
- net COL3_R: track 138.8 -> 131.4 mm, vias 7 -> 9
- net GND: track 30.2 -> 23.2 mm
- net Net-(D9-A): track 11.9 -> 6.86 mm
- net ROW1_R: track 138.5 -> 133.6 mm
- net COL5_L: track 71.0 -> 75.9 mm, vias 5 -> 7
- net ROW0_R: track 127.1 -> 122.7 mm
- net COL4_L: track 143.9 -> 147.4 mm
- net VBAT_R: track 42.9 -> 40.0 mm
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Other:
- outline, holes or cut-outs redrawn
