File: rev1/PCB/corne-xiao-backups/backup/corne-xiao.kicad_sch (KiCad schematic)
At the start: 104 parts, among them SW1 SW_PUSH, SW10 SW_PUSH, SW11 SW_PUSH, SW12 SW_PUSH, SW13 SW_PUSH, SW14 SW_PUSH, SW15 SW_PUSH, SW16 SW_PUSH, SW17 SW_PUSH, SW18 SW_PUSH, SW19 SW_PUSH, SW2 SW_PUSH, SW20 SW_PUSH, SW21 SW_PUSH, SW22 SW_PUSH, SW23 SW_PUSH, SW24 SW_PUSH, SW25 SW_PUSH, SW26 SW_PUSH, SW27 SW_PUSH, SW28 SW_PUSH, SW29 SW_PUSH, SW3 SW_PUSH, SW30 SW_PUSH, SW31 SW_PUSH, SW32 SW_PUSH, SW33 SW_PUSH, SW34 SW_PUSH, SW35 SW_PUSH, SW36 SW_PUSH, SW37 SW_PUSH, SW38 SW_PUSH, SW39 SW_PUSH, SW4 SW_PUSH, SW40 SW_PUSH, SW41 SW_PUSH, SW42 SW_PUSH, SW5 SW_PUSH, SW6 SW_PUSH, SW7 SW_PUSH, SW8 SW_PUSH, SW9 SW_PUSH, U1 xiao-ble, U2 xiao-ble

Commit message: Backup
Parts:
- D1, D10, D11, D12, D13, D14, D15, D16, D17, D18, D19, D2, D20, D21, D22, D23, D24, D25, D26, D27, D28, D29, D3, D30, D31, D32, D33, D34, D35, D36, D37, D38, D39, D4, D40, D41, D42, D5, D6, D7, D8, D9: footprint ScottoKeebs_Components:Diode_SOD-123 -> kbd:D3_SMD_v2
Changed lines of the file:
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@@
 			)
 		)
-		(property "Footprint" "ScottoKeebs_Components:Diode_SOD-123"
+		(property "Footprint" "kbd:D3_SMD_v2"
 			(at 99.06 133.096 0)
 			(effects
@@
 			)
 		)
-		(property "Footprint" "ScottoKeebs_Components:Diode_SOD-123"
+		(property "Footprint" "kbd:D3_SMD_v2"
 			(at 116.84 133.096 0)
 			(effects
@@
 			)
 		)
-		(property "Footprint" "ScottoKeebs_Components:Diode_SOD-123"
+		(property "Footprint" "kbd:D3_SMD_v2"
 			(at 134.62 133.096 0)
 			(effects
@@
 			)
 		)
-		(property "Footprint" "ScottoKeebs_Components:Diode_SOD-123"
+		(property "Footprint" "kbd:D3_SMD_v2"
 			(at 152.4 133.096 0)
 			(effects
@@
 			)
 		)
-		(property "Footprint" "ScottoKeebs_Components:Diode_SOD-123"
+		(property "Footprint" "kbd:D3_SMD_v2"
 			(at 170.18 133.096 0)
 			(effects
@@
 			)
 		)
-		(property "Footprint" "ScottoKeebs_Components:Diode_SOD-123"
+		(property "Footprint" "kbd:D3_SMD_v2"
 			(at 81.28 133.096 0)
 			(effects
@@
 			)
 		)
-		(property "Footprint" "ScottoKeebs_Components:Diode_SOD-123"
+		(property "Footprint" "kbd:D3_SMD_v2"
 			(at 99.06 148.336 0)
 			(effects
@@
 			)
 		)
-		(property "Footprint" "ScottoKeebs_Components:Diode_SOD-123"
+		(property "Footprint" "kbd:D3_SMD_v2"
 			(at 116.84 148.336 0)
 			(effects
@@
 			)
 		)
-		(property "Footprint" "ScottoKeebs_Components:Diode_SOD-123"
+		(property "Footprint" "kbd:D3_SMD_v2"
 			(at 134.62 148.336 0)
 			(effects
@@
 			)
 		)
-		(property "Footprint" "ScottoKeebs_Components:Diode_SOD-123"
+		(property "Footprint" "kbd:D3_SMD_v2"
 			(at 152.4 148.336 0)
 			(effects
@@
 			)
 		)
-		(property "Footprint" "ScottoKeebs_Components:Diode_SOD-123"
+		(property "Footprint" "kbd:D3_SMD_v2"
 			(at 170.18 148.336 0)
 			(effects
@@
 			)
 		)
-		(property "Footprint" "ScottoKeebs_Components:Diode_SOD-123"
+		(property "Footprint" "kbd:D3_SMD_v2"
 			(at 81.28 148.336 0)
 			(effects
@@
 			)
 		)
-		(property "Footprint" "ScottoKeebs_Components:Diode_SOD-123"
+		(property "Footprint" "kbd:D3_SMD_v2"
 			(at 99.06 163.576 0)
 			(effects
@@
 			)
 		)
-		(property "Footprint" "ScottoKeebs_Components:Diode_SOD-123"
+		(property "Footprint" "kbd:D3_SMD_v2"
 			(at 116.84 163.576 0)
 			(effects
@@
 			)
 		)
-		(property "Footprint" "ScottoKeebs_Components:Diode_SOD-123"
+		(property "Footprint" "kbd:D3_SMD_v2"
 			(at 134.62 163.576 0)
 			(effects
@@
 			)
 		)
-		(property "Footprint" "ScottoKeebs_Components:Diode_SOD-123"
+		(property "Footprint" "kbd:D3_SMD_v2"
 			(at 152.4 163.576 0)
 			(effects
@@
 			)
 		)
-		(property "Footprint" "ScottoKeebs_Components:Diode_SOD-123"
+		(property "Footprint" "kbd:D3_SMD_v2"
 			(at 170.18 163.576 0)
 			(effects
@@
 			)
 		)
-		(property "Footprint" "ScottoKeebs_Components:Diode_SOD-123"
+		(property "Footprint" "kbd:D3_SMD_v2"
 			(at 81.28 163.576 0)
 			(effects
@@
 			)
 		)
-		(property "Footprint" "ScottoKeebs_Components:Diode_SOD-123"
+		(property "Footprint" "kbd:D3_SMD_v2"
 			(at 134.62 178.816 0)
 			(effects
@@
 			)
 		)
-		(property "Footprint" "ScottoKeebs_Components:Diode_SOD-123"
+		(property "Footprint" "kbd:D3_SMD_v2"
 			(at 152.4 178.816 0)
 			(effects
@@
 			)
 		)
-		(property "Footprint" "ScottoKeebs_Components:Diode_SOD-123"
+		(property "Footprint" "kbd:D3_SMD_v2"
 			(at 116.84 178.816 0)
 			(effects
@@
 			)
 		)
-		(property "Footprint" "ScottoKeebs_Components:Diode_SOD-123"
+		(property "Footprint" "kbd:D3_SMD_v2"
 			(at 281.94 133.096 0)
 			(effects
@@
 			)
 		)
-		(property "Footprint" "ScottoKeebs_Components:Diode_SOD-123"
+		(property "Footprint" "kbd:D3_SMD_v2"
 			(at 299.72 133.096 0)
 			(effects
@@
 			)
 		)
-		(property "Footprint" "ScottoKeebs_Components:Diode_SOD-123"
+		(property "Footprint" "kbd:D3_SMD_v2"
 			(at 317.5 133.096 0)
 			(effects
@@
 			)
 		)
-		(property "Footprint" "ScottoKeebs_Components:Diode_SOD-123"
+		(property "Footprint" "kbd:D3_SMD_v2"
 			(at 335.28 133.096 0)
 			(effects
@@
 			)
 		)
-		(property "Footprint" "ScottoKeebs_Components:Diode_SOD-123"
+		(property "Footprint" "kbd:D3_SMD_v2"
 			(at 353.06 133.096 0)
 			(effects
@@
 			)
 		)
-		(property "Footprint" "ScottoKeebs_Components:Diode_SOD-123"
+		(property "Footprint" "kbd:D3_SMD_v2"
 			(at 264.16 133.096 0)
 			(effects
@@
 			)
 		)
-		(property "Footprint" "ScottoKeebs_Components:Diode_SOD-123"
+		(property "Footprint" "kbd:D3_SMD_v2"
 			(at 281.94 148.336 0)
 			(effects
@@
 			)
 		)
-		(property "Footprint" "ScottoKeebs_Components:Diode_SOD-123"
+		(property "Footprint" "kbd:D3_SMD_v2"
 			(at 299.72 148.336 0)
 			(effects
@@
 			)
 		)
-		(property "Footprint" "ScottoKeebs_Components:Diode_SOD-123"
+		(property "Footprint" "kbd:D3_SMD_v2"
 			(at 317.5 148.336 0)
 			(effects
@@
 			)
 		)
-		(property "Footprint" "ScottoKeebs_Components:Diode_SOD-123"
+		(property "Footprint" "kbd:D3_SMD_v2"
 			(at 335.28 148.336 0)
 			(effects
@@
 			)
 		)
-		(property "Footprint" "ScottoKeebs_Components:Diode_SOD-123"
+		(property "Footprint" "kbd:D3_SMD_v2"
 			(at 353.06 148.336 0)
 			(effects
@@
 			)
 		)
-		(property "Footprint" "ScottoKeebs_Components:Diode_SOD-123"
+		(property "Footprint" "kbd:D3_SMD_v2"
 			(at 264.16 148.336 0)
 			(effects
@@
 			)
 		)
-		(property "Footprint" "ScottoKeebs_Components:Diode_SOD-123"
+		(property "Footprint" "kbd:D3_SMD_v2"
 			(at 281.94 163.576 0)
 			(effects
@@
 			)
 		)
-		(property "Footprint" "ScottoKeebs_Components:Diode_SOD-123"
+		(property "Footprint" "kbd:D3_SMD_v2"
 			(at 299.72 163.576 0)
 			(effects
@@
 			)
 		)
-		(property "Footprint" "ScottoKeebs_Components:Diode_SOD-123"
+		(property "Footprint" "kbd:D3_SMD_v2"
 			(at 317.5 163.576 0)
 			(effects
@@
 			)
 		)
-		(property "Footprint" "ScottoKeebs_Components:Diode_SOD-123"
+		(property "Footprint" "kbd:D3_SMD_v2"
 			(at 335.28 163.576 0)
 			(effects
@@
 			)
 		)
-		(property "Footprint" "ScottoKeebs_Components:Diode_SOD-123"
+		(property "Footprint" "kbd:D3_SMD_v2"
 			(at 353.06 163.576 0)
 			(effects
@@
 			)
 		)
-		(property "Footprint" "ScottoKeebs_Components:Diode_SOD-123"
+		(property "Footprint" "kbd:D3_SMD_v2"
 			(at 264.16 163.576 0)
 			(effects
@@
 			)
 		)
-		(property "Footprint" "ScottoKeebs_Components:Diode_SOD-123"
+		(property "Footprint" "kbd:D3_SMD_v2"
 			(at 317.5 178.816 0)
 			(effects
@@
 			)
 		)
-		(property "Footprint" "ScottoKeebs_Components:Diode_SOD-123"
+		(property "Footprint" "kbd:D3_SMD_v2"
 			(at 335.28 178.816 0)
 			(effects
@@
 			)
 		)
-		(property "Footprint" "ScottoKeebs_Components:Diode_SOD-123"
+		(property "Footprint" "kbd:D3_SMD_v2"
 			(at 299.72 178.816 0)
 			(effects
